File: PCB_layout/miniPIC/miniPIC.kicad_pcb (KiCad board)
At the start: 2 copper layers, 77.4 x 65.2 mm, 45 parts, among them J1 Conn_01x09, J2 Conn_01x06, J3 Conn_01x10, J4 Conn_01x08, J5 Jack-DC, J6 Conn_01x05, J7 Conn_01x04, J9 USB_B_Mini, SW1 EG2201B, U1 PIC16F887-IP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

Commit message: add: PCB_layout
Parts:
- moved C1 2.19 mm to (118.9, 76.6)
- moved C3 1.91 mm to (114.0, 76.7)
Routing:
- net /RA6: track 15.3 -> 13.1 mm
- net /RA7: track 14.1 -> 12.1 mm
Changed lines of the file:
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@@
 			(crossoutdnponfab yes)
 			(subtractmaskfromsilk no)
-			(outputformat 1)
+			(outputformat 4)
 			(mirror no)
-			(drillshape 1)
+			(drillshape 0)
 			(scaleselection 1)
-			(outputdirectory "")
+			(outputdirectory "C:/Users/PC/Downloads/")
 		)
 	)
@@
 		)
 		(property "Value" "Crystal"
-			(at 2.44 3.52 0)
+			(at 11.48 0.14 0)
 			(layer "F.Fab")
 			(effects
@@
 	(footprint "Capacitor_Tantalum_SMD:CP_EIA-1608-08_AVX-J"
 		(layer "F.Cu")
-		(at 120.495 75.1)
+		(at 118.9125 76.62)
 		(descr "Tantalum Capacitor SMD AVX-J (1608-08 Metric), IPC-7352 nominal, (Body size from: https://www.vishay.com/docs/48064/_t58_vmn_pt0471_1601.pdf), generated with kicad-footprint-generator")
 		(tags "capacitor tantalum")
@@
 		)
 		(property "Value" "22pF"
-			(at 0 1.52 0)
+			(at 3.5475 0.06 0)
 			(layer "F.Fab")
 			(effects
@@
 	(footprint "Capacitor_Tantalum_SMD:CP_EIA-1608-08_AVX-J"
 		(layer "F.Cu")
-		(at 114.65 74.85)
+		(at 114 76.65)
 		(descr "Tantalum Capacitor SMD AVX-J (1608-08 Metric), IPC-7352 nominal, (Body size from: https://www.vishay.com/docs/48064/_t58_vmn_pt0471_1601.pdf), generated with kicad-footprint-generator")
 		(tags "capacitor tantalum")
@@
 		)
 		(property "Value" "22pF"
-			(at 0 1.52 0)
+			(at -3.56 0 0)
 			(layer "F.Fab")
 			(effects
@@
 		(model "${KICAD9_3DMODEL_DIR}/MCU.3dshapes/PIC16F887-I_P.step"
 			(offset
-				(xyz 0 0 7)
+				(xyz 0 0 -8)
 			)
 			(scale
@@
 	)
 	(segment
-		(start 110.42 83.57)
-		(end 113.11 80.88)
-		(width 0.4)
-		(layer "F.Cu")
-		(net 7)
-	)
-	(segment
-		(start 113.11 80.88)
-		(end 113.11 76.07)
+		(start 113.285 76.65)
+		(end 113.285 80.705)
 		(width 0.4)
 		(layer "F.Cu")
@@
 	)
 	(segment
-		(start 113.935 75.245)
-		(end 113.11 76.07)
+		(start 110.42 83.57)
+		(end 113.11 80.88)
 		(width 0.4)
 		(layer "F.Cu")
@@
 	)
 	(segment
-		(start 113.935 74.85)
-		(end 113.935 75.245)
+		(start 113.285 80.705)
+		(end 113.11 80.88)
 		(width 0.4)
 		(layer "F.Cu")
@@
 	)
 	(segment
-		(start 119.78 79.09)
-		(end 117.99 80.88)
+		(start 117.99 80.88)
+		(end 117.99 82.4955)
 		(width 0.4)
 		(layer "F.Cu")
@@
 	)
 	(segment
-		(start 117.99 80.88)
-		(end 117.99 82.4955)
+		(start 118.1975 80.6725)
+		(end 117.99 80.88)
 		(width 0.4)
 		(layer "F.Cu")
@@
 	)
 	(segment
-		(start 119.78 75.1)
-		(end 119.78 79.09)
+		(start 118.1975 76.62)
+		(end 118.1975 80.6725)
 		(width 0.4)
 		(layer "F.Cu")
